File: STM32_DVM_C3ROC.sch (KiCad schematic (older format))
At the start: 31 parts, among them J1 40HAT, Q1 DMG2305UX, Q2 DMMT5401, U3 MCP6002-xSN

Commit message: Schaltplan bis auf USB und DC/DC komplett
Parts:
- removed Q1: DMG2305UX, Package_TO_SOT_SMD:SOT-23, symbol raspberrypi_hat:DMG2305UX
- removed Q2: DMMT5401, Package_TO_SOT_SMD:SOT-23-6, symbol raspberrypi_hat:DMMT5401
- removed R23: 10K, Resistor_SMD:R_0603_1608Metric_Pad0.84x1.00mm_HandSolder, symbol Device:R
- removed U? (x2): MCP6002-xSN, symbol Amplifier_Operational:MCP6002-xSN
- added C11, C28, C32, C35, C4, C8, C9, C?: 4u7, symbol Device:C
- added C12, C13: 10p, symbol Device:C
- added C14, C19, C20, C33, C34: 22u, symbol Device:C
- added C15, C17, C22: 47u, symbol Device:C
- added C2, C5, C7, C? (x5): 100n, symbol Device:C
- added C24, C27, C?: 10n, symbol Device:C
- added C29: 680p, symbol Device:C
- added C?: 1u, symbol Device:C
- added D1: BAV70, Package_TO_SOT_SMD:SOT-23, symbol Diode:BAV70
- added FB1, FB? (x22): 100, symbol Device:Ferrite_Bead
- added unit 1 of IC2
- added unit 2 of IC2
- added JP2: Nextion Display, symbol Connector_Generic:Conn_01x04
- added JP3: Debug, symbol Connector_Generic:Conn_02x03_Odd_Even
- added JP4: To LED + Display, symbol Connector_Generic:Conn_02x10_Odd_Even
- added JP5: To STM32 DVM, symbol Connector_Generic:Conn_02x10_Odd_Even
- added JP?: I2C Display, symbol Connector_Generic:Conn_01x04
- added LED1, LED6: RED, symbol Device:LED
- added LED10, LED11, LED7, LED8, LED9: YEL, symbol Device:LED
- added LED12: VIO, symbol Device:LED
- added LED2: BLU, symbol Device:LED
- added LED3, LED4: ORG, symbol Device:LED
- added LED5: GRN, symbol Device:LED
- added Q1: Crystal_GND23, symbol Device:Crystal_GND23
- added R1, R2, R34, R36, R41: 1k, Resistor_SMD:R_0603_1608Metric_Pad0.84x1.00mm_HandSolder, symbol Device:R
- added R10, R4, R?: 10K, Resistor_SMD:R_0603_1608Metric_Pad0.84x1.00mm_HandSolder, symbol Device:R
- added R11, R12, R13, R14: 22k, Resistor_SMD:R_0603_1608Metric_Pad0.84x1.00mm_HandSolder, symbol Device:R
- added R15, R16, R21: 100k, Resistor_SMD:R_0603_1608Metric_Pad0.84x1.00mm_HandSolder, symbol Device:R
- added R20: 68k, Resistor_SMD:R_0603_1608Metric_Pad0.84x1.00mm_HandSolder, symbol Device:R
- added R22: 3k3, Resistor_SMD:R_0603_1608Metric_Pad0.84x1.00mm_HandSolder, symbol Device:R
- added R26: 3k9, Resistor_SMD:R_0603_1608Metric_Pad0.84x1.00mm_HandSolder, symbol Device:R
- added R29, R31, R37, R?: 47, Resistor_SMD:R_0603_1608Metric_Pad0.84x1.00mm_HandSolder, symbol Device:R
- added R30: 47k, Resistor_SMD:R_0603_1608Metric_Pad0.84x1.00mm_HandSolder, symbol Device:R
- added R32: 10k, symbol Device:R_POT_TRIM
- added R33, R35, R5, R8: 10k, Resistor_SMD:R_0603_1608Metric_Pad0.84x1.00mm_HandSolder, symbol Device:R
- added R39: 4k7, Resistor_SMD:R_0603_1608Metric_Pad0.84x1.00mm_HandSolder, symbol Device:R
- added R42, R43, R44, R45, R46, R47, R48, R49, R50, R?: 560, Resistor_SMD:R_0603_1608Metric_Pad0.84x1.00mm_HandSolder, symbol Device:R
- added R6: 100k, symbol Device:R_POT_TRIM
- added R7: 100, Resistor_SMD:R_0603_1608Metric_Pad0.84x1.00mm_HandSolder, symbol Device:R
- added SJ1: Jumper_2_Open, symbol Jumper:Jumper_2_Open
- added SW?: SW_Push, symbol Switch:SW_Push
- added T1, T2, T3, T4: MMUN2214, symbol Device:Q_NPN_BEC_BRT
- added TP1, TP2, TP5: TestPoint, symbol Connector:TestPoint
- added TP3: RXA, symbol Connector:TestPoint
- added TP6: TXA_R, symbol Connector:TestPoint
- added TP7: RSSI, symbol Connector:TestPoint
- added U?: TPS54360DDA, Package_SO:TI_SO-PowerPAD-8_ThermalVias, symbol Regulator_Switching:TPS54360DDA
- added X?: ASE-12MHz, Oscillator:Oscillator_SMD_Abracon_ASE-4Pin_3.2x2.5mm, symbol Oscillator:ASE-xxxMHz
- C31: renamed from C?; value 10n -> 680p
- C?: value C -> 1u
- H1, H2, H3, H4: value 3mm_Mounting_Hole -> 3mm
- IC2, IC4: renamed from U?; value MCP6002-xSN -> MCP6002
- IC3: renamed from U3; value MCP6002-xSN -> MCP6002
- R19: renamed from R?; value 10K -> 10k
- R23: renamed from RV23; value 100K -> 100k
- R24: value 47K -> 39k
- R38: renamed from R?; value 10K -> 47k
- R51: renamed from RV?; value R_POT_TRIM -> 100k
- X2: renamed from J?; value DB9_Female_MountingHoles -> To Radio
- gave numbers to parts that had none: 2
Connections:
- net labels added: +3.3VA, BOOT0, GNDA, INHIBIT_R, INIHIBIT_R, LED_CLIP, NRST, PTT_R, RSSI_R, RXA_R, SR_RX, SR_TX, TXA_R
- net labels removed: P3V3_HAT, P5V, P5V_HAT
- wire segments 78 -> 437
Other:
- note added: "Cut off LED and Display Connection"
- moved on the sheet: C21, C26, C30, C31, C?, H1, H2, H3, H4, IC2C, IC3A, IC3B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

Commit message: Schaltplan fertig, Footprints zugewiesen, PCB Beginn platzierung
Parts:
- added C23, C25: 2u2, Capacitor_SMD:C_1206_3216Metric, symbol Device:C
- added C36: 6n8, Capacitor_SMD:C_0603_1608Metric, symbol Device:C
- added C37: 47p, Capacitor_SMD:C_0603_1608Metric, symbol Device:C
- added C38: 100n, Capacitor_SMD:C_0603_1608Metric, symbol Device:C
- added C39, C40: 22u, Capacitor_SMD:C_1206_3216Metric, symbol Device:C
- added D2: B560C, Diode_SMD:D_SMC, symbol Device:D_Schottky
- added J2: USB_B_Micro, Connector_USB:USB_Micro-B_Molex_47346-0001, symbol Connector:USB_B_Micro
- added L1: 8u2, Inductor_SMD:L_Coilcraft_XAL60xx_6.36x6.56mm, symbol Device:L
- added R18, R40: 10k, Resistor_SMD:R_0603_1608Metric, symbol Device:R
- added R52: 162k, Resistor_SMD:R_0603_1608Metric, symbol Device:R
- added R53, R55: 10k2, Resistor_SMD:R_0603_1608Metric, symbol Device:R
- added R54: 53k6, Resistor_SMD:R_0603_1608Metric, symbol Device:R
- added U2, U3, U4: USBLC6-2SC6, Package_TO_SOT_SMD:SOT-23-6, symbol Power_Protection:USBLC6-2SC6
- C1, C10, C16, C3, C42, C6: renamed from C?; footprint (none) -> Capacitor_SMD:C_0603_1608Metric
- C11, C28, C32, C35, C4, C8, C9: footprint (none) -> Capacitor_SMD:C_1206_3216Metric
- C12, C13, C2, C24, C26, C27, C29, C30, C31, C5, C7: footprint (none) -> Capacitor_SMD:C_0603_1608Metric
- C14, C15, C17, C19, C20, C21, C22, C33, C34: footprint (none) -> Capacitor_SMD:C_1210_3225Metric
- C18, C41, C43: renamed from C?; footprint (none) -> Capacitor_SMD:C_1206_3216Metric
- FB1: footprint (none) -> Inductor_SMD:L_0603_1608Metric
- FB10, FB11, FB12, FB13, FB14, FB15, FB16, FB17, FB18, FB19, FB2, FB20, FB21, FB22, FB23, FB3, FB4, FB5, FB6, FB7, FB8, FB9: renamed from FB?; footprint (none) -> Inductor_SMD:L_0603_1608Metric
- IC2, IC3, IC4: footprint (none) -> Package_SO:SO-8_3.9x4.9mm_P1.27mm
- JP1: renamed from JP?; footprint (none) -> Connector_PinHeader_2.54mm:PinHeader_1x04_P2.54mm_Vertical
- JP2: footprint (none) -> Connector_PinHeader_2.54mm:PinHeader_1x04_P2.54mm_Vertical
- JP3: footprint (none) -> Connector_PinHeader_2.54mm:PinHeader_2x03_P2.54mm_Vertical
- JP4, JP5: footprint (none) -> Connector_PinHeader_2.54mm:PinHeader_2x10_P2.54mm_Vertical
- LED1, LED10, LED11, LED12, LED2, LED3, LED4, LED5, LED6, LED7, LED8, LED9: footprint (none) -> LED_SMD:LED_0603_1608Metric
- Q1: footprint (none) -> Crystal:Crystal_SMD_3225-4Pin_3.2x2.5mm
- R1, R10, R11, R12, R13, R14, R15, R16, R19, R2, R20, R21, R22, R24, R25, R26, R27, R28, R29, R3, R30, R31, R33, R34, R35, R36, R37, R38, R39, R4, R41, R42, R43, R44, R45, R46, R47, R48, R49, R5, R50, R7, R8: footprint Resistor_SMD:R_0603_1608Metric_Pad0.84x1.00mm_HandSolder -> Resistor_SMD:R_0603_1608Metric
- R17, R56, R9: renamed from R?; footprint Resistor_SMD:R_0603_1608Metric_Pad0.84x1.00mm_HandSolder -> Resistor_SMD:R_0603_1608Metric
- R23, R32, R51, R6: footprint (none) -> Resistor_SMD:R_0603_1608Metric
- SJ1: footprint (none) -> Jumper:SolderJumper-2_P1.3mm_Open_Pad1.0x1.5mm
- T1, T2, T3, T4: footprint (none) -> Package_TO_SOT_SMD:SOT-23
- TP1, TP2, TP3, TP5, TP6, TP7: footprint (none) -> TestPoint:TestPoint_Pad_1.5x1.5mm
- X2: footprint (none) -> Connector_Dsub:DSUB-9_Female_Vertical_P2.77x2.84mm_MountingHoles
- gave numbers to parts that had none: 3
Connections:
- wire segments 437 -> 489
Other:
- note removed: "40-Pin HAT Connector"
- note removed: "Mounting Holes"
- moved on the sheet: FB1, FB10, FB11, FB12, FB13, FB14, FB15, FB16, FB17, FB18, FB19, FB20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

Commit message: Zwei Fehler im Schaltplan gefixt
Connections:
- wire segments 489 -> 490
Other:
- moved on the sheet: R30
Changed lines of the file:
@@
 L Device:R R30
 U 1 1 601B865D
-P 14850 7650
-F 0 "R30" H 14700 7700 50  0000 C CNN
-F 1 "47k" H 14700 7600 50  0000 C CNN
-F 2 "Resistor_SMD:R_0603_1608Metric" V 14780 7650 50  0001 C CNN
-F 3 "" H 14850 7650 50  0001 C CNN
-	1    14850 7650
+P 14850 7750
+F 0 "R30" H 14700 7800 50  0000 C CNN
+F 1 "47k" H 14700 7700 50  0000 C CNN
+F 2 "Resistor_SMD:R_0603_1608Metric" V 14780 7750 50  0001 C CNN
+F 3 "" H 14850 7750 50  0001 C CNN
+	1    14850 7750
 	1    0    0    -1
 $EndComp
@@
 $EndComp
 Wire Wire Line
-	3800 8750 3900 8750
-Wire Wire Line
 	3450 8750 3300 8750
 Wire Wire Line
@@
 L power:GND #PWR0181
 U 1 1 63550F08
-P 14850 7900
-F 0 "#PWR0181" H 14850 7650 50  0001 C CNN
-F 1 "GND" H 14850 7750 50  0000 C CNN
-F 2 "" H 14850 7900 50  0000 C CNN
-F 3 "" H 14850 7900 50  0000 C CNN
-	1    14850 7900
-	1    0    0    -1
-$EndComp
-Text GLabel 15000 7850 2    50   Output ~ 0
+P 14850 8000
+F 0 "#PWR0181" H 14850 7750 50  0001 C CNN
+F 1 "GND" H 14850 7850 50  0000 C CNN
+F 2 "" H 14850 8000 50  0000 C CNN
+F 3 "" H 14850 8000 50  0000 C CNN
+	1    14850 8000
+	1    0    0    -1
+$EndComp
+Text GLabel 15000 7550 2    50   Output ~ 0
 INHIBIT
 $Comp
@@
 	14450 7300 14350 7300
 Wire Wire Line
-	15000 7850 14850 7850
-Wire Wire Line
-	14850 7850 14850 7900
-Wire Wire Line
-	14850 7800 14850 7850
-Connection ~ 14850 7850
+	15000 7550 14850 7550
 Text GLabel 14400 6150 0    50   Input ~ 0
 PTT_R
@@
 	1    0    0    -1
 $EndComp
+Wire Wire Line
+	3750 8750 3900 8750
+Wire Wire Line
+	14850 7900 14850 8000
+Wire Wire Line
+	14850 7550 14850 7500
+Wire Wire Line
+	14850 7600 14850 7550
+Connection ~ 14850 7550
 $EndSCHEMATC

Commit message: Etwas Bauteil Schubsen
Parts:
- U2, U3, U4: symbol Power_Protection:USBLC6-2SC6 -> STM32_DVM_C3ROC-rescue:USBLC6-2SC6-Power_Protection
Changed lines of the file:
@@
 $EndComp
 $Comp
-L Power_Protection:USBLC6-2SC6 U3
+L STM32_DVM_C3ROC-rescue:USBLC6-2SC6-Power_Protection U3
 U 1 1 5FBA17F6
 P 10500 1500
@@
 	10600 1000 10750 1000
 $Comp
-L Power_Protection:USBLC6-2SC6 U4
+L STM32_DVM_C3ROC-rescue:USBLC6-2SC6-Power_Protection U4
 U 1 1 5FE093D7
 P 10500 2750
@@
 USB_D+
 $Comp
-L Power_Protection:USBLC6-2SC6 U2
+L STM32_DVM_C3ROC-rescue:USBLC6-2SC6-Power_Protection U2
 U 1 1 60427054
 P 5000 5150

Commit message: Platzierung 90 % komplett
Parts:
- removed R17: 10K, Resistor_SMD:R_0603_1608Metric, symbol Device:R
- C11, C18, C28, C32, C8, C9: footprint Capacitor_SMD:C_1206_3216Metric -> Capacitor_SMD:C_0603_1608Metric
- R23, R32, R51, R6: footprint Resistor_SMD:R_0603_1608Metric -> Potentiometer_THT:Potentiometer_Bourns_3296W_Vertical
- SW1: footprint (none) -> Button_Switch_SMD:SW_Push_SPST_NO_Alps_SKRK
- X2: footprint Connector_Dsub:DSUB-9_Female_Vertical_P2.77x2.84mm_MountingHoles -> Connector_Dsub:DSUB-9_Female_Horizontal_P2.77x2.84mm_EdgePinOffset4.94mm_Housed_MountingHolesOffset7.48mm
Connections:
- net TXA: now also C19.1
Other:
- moved on the sheet: R8
Changed lines of the file:
@@
 EESchema Schematic File Version 4
-EELAYER 30 0
+LIBS:STM32_DVM_C3ROC-cache
+EELAYER 29 0
 EELAYER END
 $Descr A3 16535 11693
@@
 F 0 "X2" H 8430 5152 50  0000 L CNN
 F 1 "To Radio" H 8430 5061 50  0000 L CNN
-F 2 "Connector_Dsub:DSUB-9_Female_Vertical_P2.77x2.84mm_MountingHoles" H 8250 5150 50  0001 C CNN
+F 2 "Connector_Dsub:DSUB-9_Female_Horizontal_P2.77x2.84mm_EdgePinOffset4.94mm_Housed_MountingHolesOffset7.48mm" H 8250 5150 50  0001 C CNN
 F 3 " ~" H 8250 5150 50  0001 C CNN
 	1    8250 5150
@@
 F 0 "R51" H 14681 9204 50  0000 R CNN
 F 1 "100k" H 14681 9295 50  0000 R CNN
-F 2 "Resistor_SMD:R_0603_1608Metric" H 14750 9250 50  0001 C CNN
+F 2 "Potentiometer_THT:Potentiometer_Bourns_3296W_Vertical" H 14750 9250 50  0001 C CNN
 F 3 "~" H 14750 9250 50  0001 C CNN
 	1    14750 9250
@@
 F 0 "R23" H 7680 8096 50  0000 R CNN
 F 1 "100k" H 7680 8005 50  0000 R CNN
-F 2 "Resistor_SMD:R_0603_1608Metric" H 7750 8050 50  0001 C CNN
+F 2 "Potentiometer_THT:Potentiometer_Bourns_3296W_Vertical" H 7750 8050 50  0001 C CNN
 F 3 "~" H 7750 8050 50  0001 C CNN
 	1    7750 8050
@@
 F 0 "R6" H 5550 7600 50  0000 R CNN
 F 1 "100k" H 5631 7695 50  0000 R CNN
-F 2 "Resistor_SMD:R_0603_1608Metric" H 5700 7650 50  0001 C CNN
+F 2 "Potentiometer_THT:Potentiometer_Bourns_3296W_Vertical" H 5700 7650 50  0001 C CNN
 F 3 "~" H 5700 7650 50  0001 C CNN
 	1    5700 7650
@@
 F 0 "R32" H 10200 10000 50  0000 R CNN
 F 1 "10k" H 10200 10100 50  0000 R CNN
-F 2 "Resistor_SMD:R_0603_1608Metric" H 10450 9950 50  0001 C CNN
+F 2 "Potentiometer_THT:Potentiometer_Bourns_3296W_Vertical" H 10450 9950 50  0001 C CNN
 F 3 "~" H 10450 9950 50  0001 C CNN
 	1    10450 9950
@@
 L power:GND #PWR0124
 U 1 1 5FEED9FA
-P 5900 10050
-F 0 "#PWR0124" H 5900 9800 50  0001 C CNN
-F 1 "GND" H 5900 9900 50  0000 C CNN
-F 2 "" H 5900 10050 50  0000 C CNN
-F 3 "" H 5900 10050 50  0000 C CNN
-	1    5900 10050
+P 6200 10050
+F 0 "#PWR0124" H 6200 9800 50  0001 C CNN
+F 1 "GND" H 6200 9900 50  0000 C CNN
+F 2 "" H 6200 10050 50  0000 C CNN
+F 3 "" H 6200 10050 50  0000 C CNN
+	1    6200 10050
 	1    0    0    -1
 $EndComp
@@
 	6400 9050 6050 9050
 $Comp
-L Device:R R17
-U 1 1 5FEEDA36
-P 6200 9700
-F 0 "R17" V 6280 9700 50  0000 C CNN
-F 1 "10K" V 6100 9700 50  0000 C CNN
-F 2 "Resistor_SMD:R_0603_1608Metric" V 6130 9700 50  0001 C CNN
-F 3 "" H 6200 9700 50  0001 C CNN
-	1    6200 9700
-	0    -1   -1   0
-$EndComp
-$Comp
 L Device:R R8
 U 1 1 5FEEDA42
-P 5900 9900
-F 0 "R8" H 5750 9950 50  0000 C CNN
-F 1 "10k" H 5750 9850 50  0000 C CNN
-F 2 "Resistor_SMD:R_0603_1608Metric" V 5830 9900 50  0001 C CNN
-F 3 "" H 5900 9900 50  0001 C CNN
-	1    5900 9900
+P 6200 9900
+F 0 "R8" H 6050 9950 50  0000 C CNN
+F 1 "10k" H 6050 9850 50  0000 C CNN
+F 2 "Resistor_SMD:R_0603_1608Metric" V 6130 9900 50  0001 C CNN
+F 3 "" H 6200 9900 50  0001 C CNN
+	1    6200 9900
 	1    0    0    -1
 $EndComp
-Text GLabel 5700 9700 0    50   Input ~ 0
+Text GLabel 6000 9700 0    50   Input ~ 0
 TXA
 Wire Wire Line
@@
 $EndComp
 Wire Wire Line
-	5700 9700 5900 9700
+	6000 9700 6200 9700
 Wire Wire Line
-	5900 9750 5900 9700
-Connection ~ 5900 9700
+	6200 9750 6200 9700
+Connection ~ 6200 9700
 Wire Wire Line
-	5900 9700 6050 9700
+	6200 9700 6350 9700
 $Comp
 L Device:R R20
@@
 F 0 "C11" H 2700 7850 50  0000 L CNN
 F 1 "4u7" H 2700 7650 50  0000 L CNN
-F 2 "Capacitor_SMD:C_1206_3216Metric" H 2938 7600 50  0001 C CNN
+F 2 "Capacitor_SMD:C_0603_1608Metric" H 2938 7600 50  0001 C CNN
 F 3 "~" H 2900 7750 50  0001 C CNN
 	1    2900 7750
@@
 F 0 "C9" H 1050 6650 50  0000 L CNN
 F 1 "4u7" H 1050 6450 50  0000 L CNN
-F 2 "Capacitor_SMD:C_1206_3216Metric" H 1038 6400 50  0001 C CNN
+F 2 "Capacitor_SMD:C_0603_1608Metric" H 1038 6400 50  0001 C CNN
 F 3 "~" H 1000 6550 50  0001 C CNN
 	1    1000 6550
@@
 F 0 "C8" H 3150 7850 50  0000 L CNN
 F 1 "4u7" H 3150 7650 50  0000 L CNN
-F 2 "Capacitor_SMD:C_1206_3216Metric" H 3138 7600 50  0001 C CNN
+F 2 "Capacitor_SMD:C_0603_1608Metric" H 3138 7600 50  0001 C CNN
 F 3 "~" H 3100 7750 50  0001 C CNN
 	1    3100 7750
@@
 F 0 "SW1" V 4304 6948 50  0000 L CNN
 F 1 "SW_Push" V 4395 6948 50  0000 L CNN
-F 2 "" H 4350 7000 50  0001 C CNN
+F 2 "Button_Switch_SMD:SW_Push_SPST_NO_Alps_SKRK" H 4350 7000 50  0001 C CNN
 F 3 "~" H 4350 7000 50  0001 C CNN
 	1    4350 6800
@@
 F 0 "C28" H 3400 10850 50  0000 L CNN
 F 1 "4u7" H 3400 10650 50  0000 L CNN
-F 2 "Capacitor_SMD:C_1206_3216Metric" H 3638 10600 50  0001 C CNN
+F 2 "Capacitor_SMD:C_0603_1608Metric" H 3638 10600 50  0001 C CNN
 F 3 "~" H 3600 10750 50  0001 C CNN
 	1    3600 10750
@@
 F 0 "C18" H 4050 10850 50  0000 L CNN
 F 1 "4u7" H 4050 10650 50  0000 L CNN
-F 2 "Capacitor_SMD:C_1206_3216Metric" H 4288 10600 50  0001 C CNN
+F 2 "Capacitor_SMD:C_0603_1608Metric" H 4288 10600 50  0001 C CNN
 F 3 "~" H 4250 10750 50  0001 C CNN
 	1    4250 10750
@@
 F 0 "C32" H 4700 10850 50  0000 L CNN
 F 1 "4u7" H 4700 10650 50  0000 L CNN
-F 2 "Capacitor_SMD:C_1206_3216Metric" H 4938 10600 50  0001 C CNN
+F 2 "Capacitor_SMD:C_0603_1608Metric" H 4938 10600 50  0001 C CNN
 F 3 "~" H 4900 10750 50  0001 C CNN
 	1    4900 10750

Commit message: LCSC Part List angelegt, Footprints angepasst
Parts:
- removed Q1: Crystal_GND23, Crystal:Crystal_SMD_3225-4Pin_3.2x2.5mm, symbol Device:Crystal_GND23
- removed X1: ASE-12MHz, Oscillator:Oscillator_SMD_Abracon_ASE-4Pin_3.2x2.5mm, symbol Oscillator:ASE-xxxMHz
- added Q1: Crystal_GND24, Crystal:Crystal_SMD_3225-4Pin_3.2x2.5mm, symbol Device:Crystal_GND24
- added X1: IQXO-70, Oscillator:Oscillator_SMD_IQD_IQXO70-4Pin_7.5x5.0mm, symbol Oscillator:IQXO-70
- C11, C18, C28, C32, C8, C9: footprint Capacitor_SMD:C_0603_1608Metric -> Capacitor_SMD:C_1206_3216Metric
- C39, C40: footprint Capacitor_SMD:C_1206_3216Metric -> Capacitor_SMD:C_1210_3225Metric
- L1: footprint Inductor_SMD:L_Coilcraft_XAL60xx_6.36x6.56mm -> Inductor_SMD:L_Bourns_SRP7028A_7.3x6.6mm
Connections:
- net +3V3: now also X1.4 (V+)
- net GND: now also Q1.2, Q1.4, X1.2 (GND)
- net at C13.1, U1.5 (PH0): now also Q1.3
- net at C12.1, U1.6 (PH1): now also Q1.1
- net at C5.1: now also X1.3 (OUT)
Changed lines of the file:
@@
 EESchema Schematic File Version 4
-LIBS:STM32_DVM_C3ROC-cache
-EELAYER 29 0
+EELAYER 30 0
 EELAYER END
 $Descr A3 16535 11693
@@
 F 0 "C11" H 2700 7850 50  0000 L CNN
 F 1 "4u7" H 2700 7650 50  0000 L CNN
-F 2 "Capacitor_SMD:C_0603_1608Metric" H 2938 7600 50  0001 C CNN
+F 2 "Capacitor_SMD:C_1206_3216Metric" H 2938 7600 50  0001 C CNN
 F 3 "~" H 2900 7750 50  0001 C CNN
 	1    2900 7750
@@
 	3150 1500 3150 1600
 $Comp
-L Device:Crystal_GND23 Q1
-U 1 1 61E1B101
-P 3600 8750
-F 0 "Q1" H 3550 8150 50  0000 L CNN
-F 1 "Crystal_GND23" H 3350 8050 50  0000 L CNN
-F 2 "Crystal:Crystal_SMD_3225-4Pin_3.2x2.5mm" H 3600 8750 50  0001 C CNN
-F 3 "~" H 3600 8750 50  0001 C CNN
-	1    3600 8750
-	1    0    0    -1
-$EndComp
-$Comp
-L Oscillator:ASE-xxxMHz X1
-U 1 1 61E1DAB7
-P 2100 5100
-F 0 "X1" H 2450 5450 50  0000 L CNN
-F 1 "ASE-12MHz" H 2450 5350 50  0000 L CNN
-F 2 "Oscillator:Oscillator_SMD_Abracon_ASE-4Pin_3.2x2.5mm" H 2800 4750 50  0001 C CNN
-F 3 "http://www.abracon.com/Oscillators/ASV.pdf" H 2000 5100 50  0001 C CNN
-	1    2100 5100
-	1    0    0    -1
-$EndComp
-$Comp
 L power:+3.3V #PWR0155
 U 1 1 61E5E6F0
@@
 F 0 "C9" H 1050 6650 50  0000 L CNN
 F 1 "4u7" H 1050 6450 50  0000 L CNN
-F 2 "Capacitor_SMD:C_0603_1608Metric" H 1038 6400 50  0001 C CNN
+F 2 "Capacitor_SMD:C_1206_3216Metric" H 1038 6400 50  0001 C CNN
 F 3 "~" H 1000 6550 50  0001 C CNN
 	1    1000 6550
@@
 F 0 "C8" H 3150 7850 50  0000 L CNN
 F 1 "4u7" H 3150 7650 50  0000 L CNN
-F 2 "Capacitor_SMD:C_0603_1608Metric" H 3138 7600 50  0001 C CNN
+F 2 "Capacitor_SMD:C_1206_3216Metric" H 3138 7600 50  0001 C CNN
 F 3 "~" H 3100 7750 50  0001 C CNN
 	1    3100 7750
@@
 F 0 "C28" H 3400 10850 50  0000 L CNN
 F 1 "4u7" H 3400 10650 50  0000 L CNN
-F 2 "Capacitor_SMD:C_0603_1608Metric" H 3638 10600 50  0001 C CNN
+F 2 "Capacitor_SMD:C_1206_3216Metric" H 3638 10600 50  0001 C CNN
 F 3 "~" H 3600 10750 50  0001 C CNN
 	1    3600 10750
@@
 F 0 "C18" H 4050 10850 50  0000 L CNN
 F 1 "4u7" H 4050 10650 50  0000 L CNN
-F 2 "Capacitor_SMD:C_0603_1608Metric" H 4288 10600 50  0001 C CNN
+F 2 "Capacitor_SMD:C_1206_3216Metric" H 4288 10600 50  0001 C CNN
 F 3 "~" H 4250 10750 50  0001 C CNN
 	1    4250 10750
@@
 F 0 "C32" H 4700 10850 50  0000 L CNN
 F 1 "4u7" H 4700 10650 50  0000 L CNN
-F 2 "Capacitor_SMD:C_0603_1608Metric" H 4938 10600 50  0001 C CNN
+F 2 "Capacitor_SMD:C_1206_3216Metric" H 4938 10600 50  0001 C CNN
 F 3 "~" H 4900 10750 50  0001 C CNN
 	1    4900 10750
@@
 F 0 "C39" H 12450 5450 50  0000 L CNN
 F 1 "22u" H 12450 5350 50  0000 L CNN
-F 2 "Capacitor_SMD:C_1206_3216Metric" H 12788 5250 50  0001 C CNN
+F 2 "Capacitor_SMD:C_1210_3225Metric" H 12788 5250 50  0001 C CNN
 F 3 "~" H 12750 5400 50  0001 C CNN
 	1    12750 5400
@@
 F 0 "C40" H 13150 5450 50  0000 L CNN
 F 1 "22u" H 13150 5350 50  0000 L CNN
-F 2 "Capacitor_SMD:C_1206_3216Metric" H 13038 5250 50  0001 C CNN
+F 2 "Capacitor_SMD:C_1210_3225Metric" H 13038 5250 50  0001 C CNN
 F 3 "~" H 13000 5400 50  0001 C CNN
 	1    13000 5400
@@
 F 0 "L1" V 12690 5250 50  0000 C CNN
 F 1 "8u2" V 12599 5250 50  0000 C CNN
-F 2 "Inductor_SMD:L_Coilcraft_XAL60xx_6.36x6.56mm" H 12500 5250 50  0001 C CNN
+F 2 "Inductor_SMD:L_Bourns_SRP7028A_7.3x6.6mm" H 12500 5250 50  0001 C CNN
 F 3 "~" H 12500 5250 50  0001 C CNN
 	1    12500 5250
@@
 	14850 7600 14850 7550
 Connection ~ 14850 7550
+$Comp
+L Device:Crystal_GND24 Q1
+U 1 1 5FBE28A5
+P 3600 8750
+F 0 "Q1" H 3550 8150 50  0000 L CNN
+F 1 "Crystal_GND24" H 3350 8050 50  0000 L CNN
+F 2 "Crystal:Crystal_SMD_3225-4Pin_3.2x2.5mm" H 3600 8750 50  0001 C CNN
+F 3 "~" H 3600 8750 50  0001 C CNN
+	1    3600 8750
+	1    0    0    -1
+$EndComp
+$Comp
+L Oscillator:IQXO-70 X1
+U 1 1 5FC50233
+P 2100 5100
+F 0 "X1" H 2400 4800 50  0000 L CNN
+F 1 "IQXO-70" H 2300 4700 50  0000 L CNN
+F 2 "Oscillator:Oscillator_SMD_IQD_IQXO70-4Pin_7.5x5.0mm" H 2775 4775 50  0001 C CNN
+F 3 "http://www.iqdfrequencyproducts.com/products/details/iqxo-70-11-30.pdf" H 2000 5100 50  0001 C CNN
+	1    2100 5100
+	1    0    0    -1
+$EndComp
 $EndSCHEMATC
