File: STM32_DVM_C3ROC.sch (KiCad schematic (older format))
At the start: 170 parts, among them IC2 MCP6002, IC3 MCP6002, IC4 MCP6002, J1 40HAT, J2 USB_B_Micro, Q1 Crystal_GND24, SW1 SW_Push, T1 MMUN2214, T2 MMUN2214, T3 MMUN2214, T4 MMUN2214, U1 STM32F446RETx, U2 USBLC6-2SC6, U3 USBLC6-2SC6, U4 USBLC6-2SC6, U5 TPS54360DDA, X1 IQXO-70, X2 To Radio

Commit message: Layout 80 %, kleine Korrekturen
Parts:
- R10, R3, R4: value 10K -> 10k
- R18: value 10k -> 523k
- R40: value 10k -> 82k
- SW1: footprint Button_Switch_SMD:SW_Push_SPST_NO_Alps_SKRK -> Button_Switch_SMD:SW_SPST_SKQG_WithoutStem
- TP1, TP2, TP3, TP5, TP6, TP7: footprint TestPoint:TestPoint_Pad_1.5x1.5mm -> TestPoint:TestPoint_Pad_D1.5mm
Connections:
- net INIHIBIT_R is gone; now on net INHIBIT_R: FB14.2
- net PTT: now also T2.1 (B)
- net PTT_R: no longer T2.1 (B)
Changed lines of the file:
@@
 P 3900 6750
 F 0 "R3" H 4050 6800 50  0000 C CNN
-F 1 "10K" H 4100 6700 50  0000 C CNN
+F 1 "10k" H 4100 6700 50  0000 C CNN
 F 2 "Resistor_SMD:R_0603_1608Metric" V 3830 6750 50  0001 C CNN
 F 3 "" H 3900 6750 50  0001 C CNN
@@
 F 0 "TP1" H 7050 7700 50  0000 L CNN
 F 1 "TestPoint" H 7050 7600 50  0000 L CNN
-F 2 "TestPoint:TestPoint_Pad_1.5x1.5mm" H 7200 7400 50  0001 C CNN
+F 2 "TestPoint:TestPoint_Pad_D1.5mm" H 7200 7400 50  0001 C CNN
 F 3 "~" H 7200 7400 50  0001 C CNN
 	1    7000 7400
@@
 F 0 "TP2" H 7800 7050 50  0000 L CNN
 F 1 "TestPoint" H 7800 6950 50  0000 L CNN
-F 2 "TestPoint:TestPoint_Pad_1.5x1.5mm" H 7950 6750 50  0001 C CNN
+F 2 "TestPoint:TestPoint_Pad_D1.5mm" H 7950 6750 50  0001 C CNN
 F 3 "~" H 7950 6750 50  0001 C CNN
 	1    7750 6750
@@
 F 0 "TP3" H 9158 7318 50  0000 L CNN
 F 1 "RXA" H 9158 7227 50  0000 L CNN
-F 2 "TestPoint:TestPoint_Pad_1.5x1.5mm" H 9300 7200 50  0001 C CNN
+F 2 "TestPoint:TestPoint_Pad_D1.5mm" H 9300 7200 50  0001 C CNN
 F 3 "~" H 9300 7200 50  0001 C CNN
 	1    9100 7200
@@
 P 6200 7650
 F 0 "R10" V 6280 7650 50  0000 C CNN
-F 1 "10K" V 6100 7650 50  0000 C CNN
+F 1 "10k" V 6100 7650 50  0000 C CNN
 F 2 "Resistor_SMD:R_0603_1608Metric" V 6130 7650 50  0001 C CNN
 F 3 "" H 6200 7650 50  0001 C CNN
@@
 F 0 "TP5" H 7800 9750 50  0000 L CNN
 F 1 "TestPoint" H 7800 9650 50  0000 L CNN
-F 2 "TestPoint:TestPoint_Pad_1.5x1.5mm" H 7950 9450 50  0001 C CNN
+F 2 "TestPoint:TestPoint_Pad_D1.5mm" H 7950 9450 50  0001 C CNN
 F 3 "~" H 7950 9450 50  0001 C CNN
 	1    7750 9450
@@
 F 0 "TP6" H 10508 9568 50  0000 L CNN
 F 1 "TXA_R" H 10508 9477 50  0000 L CNN
-F 2 "TestPoint:TestPoint_Pad_1.5x1.5mm" H 10650 9450 50  0001 C CNN
+F 2 "TestPoint:TestPoint_Pad_D1.5mm" H 10650 9450 50  0001 C CNN
 F 3 "~" H 10650 9450 50  0001 C CNN
 	1    10450 9450
@@
 TXA_R
 Text GLabel 6850 5000 0    50   Input ~ 0
-INIHIBIT_R
+INHIBIT_R
 Text GLabel 6850 5200 0    50   Input ~ 0
 RSSI_R
@@
 P 3350 7300
 F 0 "R4" V 3450 7350 50  0000 C CNN
-F 1 "10K" V 3250 7350 50  0000 C CNN
+F 1 "10k" V 3250 7350 50  0000 C CNN
 F 2 "Resistor_SMD:R_0603_1608Metric" V 3280 7300 50  0001 C CNN
 F 3 "" H 3350 7300 50  0001 C CNN
@@
 F 0 "SW1" V 4304 6948 50  0000 L CNN
 F 1 "SW_Push" V 4395 6948 50  0000 L CNN
-F 2 "Button_Switch_SMD:SW_Push_SPST_NO_Alps_SKRK" H 4350 7000 50  0001 C CNN
+F 2 "Button_Switch_SMD:SW_SPST_SKQG_WithoutStem" H 4350 7000 50  0001 C CNN
 F 3 "~" H 4350 7000 50  0001 C CNN
 	1    4350 6800
@@
 	15000 7550 14850 7550
 Text GLabel 14400 6150 0    50   Input ~ 0
-PTT_R
+PTT
 Wire Wire Line
 	14400 6150 14500 6150
@@
 F 0 "TP7" H 14208 8918 50  0000 L CNN
 F 1 "RSSI" H 14208 8827 50  0000 L CNN
-F 2 "TestPoint:TestPoint_Pad_1.5x1.5mm" H 14350 8800 50  0001 C CNN
+F 2 "TestPoint:TestPoint_Pad_D1.5mm" H 14350 8800 50  0001 C CNN
 F 3 "~" H 14350 8800 50  0001 C CNN
 	1    14150 8800
@@
 P 10200 5800
 F 0 "R40" H 10050 5850 50  0000 C CNN
-F 1 "10k" H 10050 5750 50  0000 C CNN
+F 1 "82k" H 10050 5750 50  0000 C CNN
 F 2 "Resistor_SMD:R_0603_1608Metric" V 10130 5800 50  0001 C CNN
 F 3 "" H 10200 5800 50  0001 C CNN
@@
 P 10200 5250
 F 0 "R18" H 10050 5300 50  0000 C CNN
-F 1 "10k" H 10050 5200 50  0000 C CNN
+F 1 "523k" H 10050 5200 50  0000 C CNN
 F 2 "Resistor_SMD:R_0603_1608Metric" V 10130 5250 50  0001 C CNN
 F 3 "" H 10200 5250 50  0001 C CNN

Commit message: Layout fertig für review
Parts:
- added H5, H6, H7, H8: 3mm, project_footprints:NPTH_3mm_ID, symbol Mechanical:MountingHole
Changed lines of the file:
@@
 Wire Notes Line
 	11700 4200 11700 750
-Text Notes 13200 900  0    50   ~ 0
+Text Notes 12900 1000 0    50   ~ 0
 Cut off LED and Display Connection
 Text GLabel 6850 4800 0    50   Input ~ 0
@@
 	1    0    0    -1
 $EndComp
+$Comp
+L Mechanical:MountingHole H5
+U 1 1 5FD1BE6A
+P 14800 950
+F 0 "H5" H 14650 1050 60  0000 C CNN
+F 1 "3mm" H 14800 800 60  0000 C CNN
+F 2 "project_footprints:NPTH_3mm_ID" H 14700 950 60  0001 C CNN
+F 3 "" H 14700 950 60  0001 C CNN
+	1    14800 950
+	1    0    0    -1
+$EndComp
+$Comp
+L Mechanical:MountingHole H6
+U 1 1 5FD60DEE
+P 15100 950
+F 0 "H6" H 14950 1050 60  0000 C CNN
+F 1 "3mm" H 15100 800 60  0000 C CNN
+F 2 "project_footprints:NPTH_3mm_ID" H 15000 950 60  0001 C CNN
+F 3 "" H 15000 950 60  0001 C CNN
+	1    15100 950
+	1    0    0    -1
+$EndComp
+$Comp
+L Mechanical:MountingHole H7
+U 1 1 5FDA5D25
+P 15400 950
+F 0 "H7" H 15250 1050 60  0000 C CNN
+F 1 "3mm" H 15400 800 60  0000 C CNN
+F 2 "project_footprints:NPTH_3mm_ID" H 15300 950 60  0001 C CNN
+F 3 "" H 15300 950 60  0001 C CNN
+	1    15400 950
+	1    0    0    -1
+$EndComp
+$Comp
+L Mechanical:MountingHole H8
+U 1 1 5FDEACF1
+P 15700 950
+F 0 "H8" H 15550 1050 60  0000 C CNN
+F 1 "3mm" H 15700 800 60  0000 C CNN
+F 2 "project_footprints:NPTH_3mm_ID" H 15600 950 60  0001 C CNN
+F 3 "" H 15600 950 60  0001 C CNN
+	1    15700 950
+	1    0    0    -1
+$EndComp
